File: pcbs/bitko clock/Bitko clock.kicad_pcb (KiCad board)
At the start: 2 copper layers, 101 x 64.1 mm, 15 parts

Commit message: Moved switch to other side
Parts:
- removed the REF** at (27.9, 92.7)
- removed the REF** at (120.0, 92.7)
- removed the REF** at (120.0, 37.5)
- removed the REF** at (27.9, 37.5)
- moved BUZZ KILL SWITCH 97.5 mm to (123.2, 61.4)
- moved BRRRR 56.4 mm to (102.8, 73.4), turned to 0 degrees
- moved ? 8.35 mm to (37.4, 47.9)
- moved REF** 8.35 mm to (37.4, 38.1)
- moved ? 8.35 mm to (113.5, 47.9)
- moved JST_XH_B5B-XH-A_1x05 8.35 mm to (108.5, 38.0)
- moved MODE 8.35 mm to (71.8, 27.3)
- moved REF** 8.35 mm to (113.5, 38.1)
- moved JST_XH_B5B-XH-A_1x05 8.35 mm to (40.7, 38.1)
- moved REF** 8.35 mm to (82.4, 81.0)
- moved REF** 8.35 mm to (67.4, 81.0)
Routing:
- net (no net): track 1080.7 -> 1073.8 mm
Other:
- board text added: "+VE"
